File: JBD8-16.kicad_sch (KiCad schematic)
At the start: 52 parts, among them J1 RS232, J2 5V, SW1 RESET, U1 74LS02, U1 W65C02SxP, U10 74LS138, U11 74LS21, U12 74LS04, U13 74LS21, U14 74LS86, U15 74LS08, U16 74LS27, U17 74LS21, U18 74LS02, U19 74LS32, U2 6522, U2 74LS21, U20 74LS08, U21 74LS154, U22 74LS21, U23 74LS154, U24 74LS30, U25 74LS30, U26 74LS08, U27 74LS04, U28 74LS154, U3 28C256(ROM), U4 74LS04, U4 CY62256-70PC(RAM), U5 74LS04, U5 W65C51NxP, U6 74LS11, U6 MAX232, U7 74LS154, U8 74LS373, U9 74LS138, X1 1Mhz, Y1 1.8432Mhz

Commit message: Almost done with OS mem and reduced the complexity of many sectors uisng another decoder
Parts:
- removed unit 1 of U11
- removed U2: 74LS21, symbol 74xx:74LS21
- removed unit 3 of U2
- removed unit 2 of U2
- added unit 4 of U2
- added unit 2 of U2
- added unit 3 of U2
- added U29: 74LS30, symbol 74xx:74LS30
Connections:
- net +5V: now also U27.14 (VCC), U28.18 (E0), U28.19 (E1), U28.24 (VCC), U2.14 (VCC); no longer U17.9, U22.5
- net A11: no longer U5.1
- net A12: no longer U5.2 (CS1)
- net A13: no longer U2.24 (CS1)
- net A4: now also U28.23 (A0); no longer U15.12, U19.4, U5.9
- net A5: now also U28.22 (A1); no longer U19.5, U3.9, U5.11
- net A6: now also U28.21 (A2); no longer U19.2, U3.10
- net A7: now also U28.20 (A3); no longer U1.6, U3.11
- net A9: no longer U5.13
- net GND: now also U27.7 (GND), U28.12 (GND), U2.7 (GND)
- net H0: now also U2.3; no longer U22.1
- net H1: now also U2.4; no longer U22.2
- net H2: now also U2.5; no longer U22.4
- net H5: now also U5.13
- net HH10: now also U2.2; no longer U17.12
- net HH11: now also U2.13; no longer U17.13
- net HH9: now also U2.1; no longer U17.10
- net S0: now also U27.11
- net S15: no longer U12.9
- net at U5.10: now also U3.4
- net at U17.1, U4.1: now also U27.6; no longer U1.4
- net at U13.1, U5.6: now also U13.10
- net M0: now reaches U28.1 (S0)
- net M0: now also U27.5, U29.1
- net M9: now reaches U28.10 (S9)
- net M10: now reaches U28.11 (S10)
- net M11: now reaches U28.13 (S11)
- net M12: now reaches U28.14 (S12)
- net M13: now reaches U28.15 (S13)
- net M13: now also U5.11
- net M14: now reaches U28.16 (S14)
- net M14: now also U12.9
- net M15: now reaches U28.17 (S15)
- net M15: now also U27.9, U5.9
- net M1: now reaches U28.2 (S1)
- net M1: now also U29.2
- net M2: now reaches U28.3 (S2)
- net M2: now also U29.3
- net M3: now reaches U28.4 (S3)
- net M3: now also U29.4
- net M4: now reaches U28.5 (S4)
- net M4: now also U29.5
- net M5: now reaches U28.6 (S5)
- net M5: now also U29.6
- net M6: now reaches U28.7 (S6)
- net M6: now also U29.11
- net M7: now reaches U28.8 (S7)
- net M7: now also U29.12
- net M8: now reaches U28.9 (S8)
- net M8: now also U5.1
- net at U15.10, U20.1, U26.1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: now also U22.6
- net at U5.12: now also U13.12, U13.4, U3.3, U6.2
- net at U5.2: now also U2.10
- net at U12.3: now also U2.6; no longer U22.6
- net at U1.5: no longer U19.3
- net at U27.13: now also U2.8
- net at U2.23 (~{CS2}): no longer U5.3 (~{CS2})
- net at U13.2: now also U5.8; no longer U15.11
- net at U26.12: now also U20.8, U2.9
- net at U26.13: now also U29.8
- net at U27.10: now also U2.11
- net at U6.1: now also U12.8; no longer U15.6
- net at U19.1: no longer U19.6
- net at U13.9: now also U27.8
- net at U16.11: now also U19.3
- net at U16.9: now also U19.6
- net at U15.4: no longer U5.8
- now unconnected: U15.13, U15.5, U3.8
Other:
- note added: "Only 1 if 1100-0001-0000-0000 > 1100-0001-0111-1111"
- note added: "Only 1 if 1100-0001-1000-0000"
- note added: "Only 1 if xxxx 0101 xxxx xxxx"
- note added: "Only 1 if xxxx-xxxx-(0000-0111)-xxxx"
- note added: "Only 1 if xxxx-xxxx-1110-xxxx"
- note added: "Only 1 if xxxx-xxxx-1111-xxxx"
- note removed: "CS 0"
- note removed: "CS 1"
- note removed: "Only 1 if xxxx 0101 xxxx xxxx = 0101"
- note removed: "Only 1 if xxxx-xxxx-111x-xxxx"
- moved on the sheet: U12B, U12D, U14D, U15B, U15D, U16C, U17B, U19A, U19B, U1B, U1C, U1D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

Commit message: Worked on OS mem
Connections:
- net at U19.2: now also U14.11
Other:
- moved on the sheet: U14D
Changed lines of the file:
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@@
 	(wire
 		(pts
+			(xy 511.81 491.49) (xy 511.81 485.14)
+		)
+		(stroke
+			(width 0)
+			(type default)
+		)
+	)
+	(wire
+		(pts
 			(xy 25.4 93.98) (xy 30.48 93.98)
 		)
@@
 	(wire
 		(pts
+			(xy 511.81 485.14) (xy 581.66 485.14)
+		)
+		(stroke
+			(width 0)
+			(type default)
+		)
+	)
+	(wire
+		(pts
 			(xy 322.58 285.75) (xy 327.66 285.75)
 		)
@@
 	(wire
 		(pts
+			(xy 581.66 485.14) (xy 581.66 487.68)
+		)
+		(stroke
+			(width 0)
+			(type default)
+		)
+	)
+	(wire
+		(pts
+			(xy 563.88 494.03) (xy 612.14 494.03)
+		)
+		(stroke
+			(width 0)
+			(type default)
+		)
+	)
+	(wire
+		(pts
 			(xy 403.86 434.34) (xy 403.86 353.06)
 		)
@@
 	(wire
 		(pts
+			(xy 581.66 487.68) (xy 612.14 487.68)
+		)
+		(stroke
+			(width 0)
+			(type default)
+		)
+	)
+	(wire
+		(pts
 			(xy 373.38 223.52) (xy 463.55 223.52)
 		)
@@
 		)
 	)
+	(wire
+		(pts
+			(xy 529.59 596.9) (xy 590.55 596.9)
+		)
+		(stroke
+			(width 0)
+			(type default)
+		)
+	)
 	(bus
 		(pts
@@
 	(wire
 		(pts
+			(xy 554.99 619.76) (xy 590.55 619.76)
+		)
+		(stroke
+			(width 0)
+			(type default)
+		)
+	)
+	(wire
+		(pts
 			(xy 453.39 175.26) (xy 481.33 175.26)
 		)
@@
 		)
 	)
+	(wire
+		(pts
+			(xy 508 568.96) (xy 612.14 568.96)
+		)
+		(stroke
+			(width 0)
+			(type default)
+		)
+	)
 	(bus
 		(pts
@@
 	(text "Only 1 if 1100-0001-1000-0000"
 		(exclude_from_sim no)
-		(at 538.48 614.172 0)
+		(at 553.974 613.918 0)
 		(effects
 			(font
@@
 	(label "A6"
 		(at 314.96 548.64 0)
+		(fields_autoplaced yes)
 		(effects
 			(font
@@
 	(label "M15"
 		(at 186.69 464.82 0)
+		(fields_autoplaced yes)
 		(effects
 			(font
@@
 	(label "M3"
 		(at 487.68 609.6 0)
+		(fields_autoplaced yes)
 		(effects
 			(font
@@
 	(label "M3"
 		(at 271.78 546.1 0)
+		(fields_autoplaced yes)
 		(effects
 			(font
@@
 	(label "M8"
 		(at 487.68 624.84 0)
+		(fields_autoplaced yes)
 		(effects
 			(font
@@
 	(label "H5"
 		(at 307.34 416.56 0)
+		(fields_autoplaced yes)
 		(effects
 			(font
@@
 	(label "M5"
 		(at 487.68 614.68 0)
+		(fields_autoplaced yes)
 		(effects
 			(font
@@
 	(label "M4"
 		(at 487.68 612.14 0)
+		(fields_autoplaced yes)
 		(effects
 			(font
@@
 	(label "A5"
 		(at 314.96 551.18 0)
+		(fields_autoplaced yes)
 		(effects
 			(font
@@
 	(label "M1"
 		(at 487.68 604.52 0)
+		(fields_autoplaced yes)
 		(effects
 			(font
@@
 	(label "M12"
 		(at 271.78 523.24 0)
+		(fields_autoplaced yes)
 		(effects
 			(font
@@
 	(label "A4"
 		(at 314.96 553.72 0)
+		(fields_autoplaced yes)
 		(effects
 			(font
@@
 	(label "M7"
 		(at 271.78 535.94 0)
+		(fields_autoplaced yes)
 		(effects
 			(font
@@
 	(label "M0"
 		(at 487.68 601.98 0)
+		(fields_autoplaced yes)
 		(effects
 			(font
@@
 	(label "M9"
 		(at 271.78 530.86 0)
+		(fields_autoplaced yes)
 		(effects
 			(font
@@
 	(label "M0"
 		(at 271.78 553.72 0)
+		(fields_autoplaced yes)
 		(effects
 			(font
@@
 	(label "M14"
 		(at 186.69 449.58 0)
+		(fields_autoplaced yes)
 		(effects
 			(font
@@
 	(label "M2"
 		(at 487.68 607.06 0)
+		(fields_autoplaced yes)
 		(effects
 			(font
@@
 	(label "M13"
 		(at 271.78 520.7 0)
+		(fields_autoplaced yes)
 		(effects
 			(font
@@
 	(label "M8"
 		(at 271.78 533.4 0)
+		(fields_autoplaced yes)
 		(effects
 			(font
@@
 	(label "M4"
 		(at 271.78 543.56 0)
+		(fields_autoplaced yes)
 		(effects
 			(font
@@
 	(label "M0"
 		(at 231.14 532.13 0)
+		(fields_autoplaced yes)
 		(effects
 			(font
@@
 	(label "M10"
 		(at 271.78 528.32 0)
+		(fields_autoplaced yes)
 		(effects
 			(font
@@
 	(label "M14"
 		(at 271.78 518.16 0)
+		(fields_autoplaced yes)
 		(effects
 			(font
@@
 	(label "S0"
 		(at 487.68 633.73 0)
+		(fields_autoplaced yes)
 		(effects
 			(font
@@
 	(label "M5"
 		(at 271.78 541.02 0)
+		(fields_autoplaced yes)
 		(effects
 			(font
@@
 	(label "M15"
 		(at 271.78 515.62 0)
+		(fields_autoplaced yes)
 		(effects
 			(font
@@
 	(label "M7"
 		(at 487.68 619.76 0)
+		(fields_autoplaced yes)
 		(effects
 			(font
@@
 	(label "A7"
 		(at 314.96 546.1 0)
+		(fields_autoplaced yes)
 		(effects
 			(font
@@
 	(label "M13"
 		(at 298.45 402.59 0)
+		(fields_autoplaced yes)
 		(effects
 			(font
@@
 	(label "M15"
 		(at 118.11 486.41 0)
+		(fields_autoplaced yes)
 		(effects
 			(font
@@
 	(label "M6"
 		(at 271.78 538.48 0)
+		(fields_autoplaced yes)
 		(effects
 			(font
@@
 	(label "M1"
 		(at 271.78 551.18 0)
+		(fields_autoplaced yes)
 		(effects
 			(font
@@
 	(label "M2"
 		(at 271.78 548.64 0)
+		(fields_autoplaced yes)
 		(effects
 			(font
@@
 	(label "M11"
 		(at 271.78 525.78 0)
+		(fields_autoplaced yes)
 		(effects
 			(font
@@
 	(label "M6"
 		(at 487.68 617.22 0)
+		(fields_autoplaced yes)
 		(effects
 			(font
@@
 	(symbol
 		(lib_id "74xx:74LS86")
-		(at 694.69 336.55 180)
+		(at 690.88 405.13 0)
 		(unit 4)
 		(exclude_from_sim no)
@@
 		(dnp no)
 		(property "Reference" "U14"
-			(at 695.452 337.82 0)
+			(at 690.118 403.86 0)
 			(effects
 				(font
@@
 		)
 		(property "Value" "74LS86"
-			(at 695.452 335.28 0)
+			(at 690.118 406.4 0)
 			(effects
 				(font
@@
 		)
 		(property "Footprint" ""
-			(at 694.69 336.55 0)
+			(at 690.88 405.13 0)
 			(effects
 				(font
@@
 		)
 		(property "Datasheet" "74xx/74ls86.pdf"
-			(at 694.69 336.55 0)
+			(at 690.88 405.13 0)
 			(effects
 				(font
@@
 		)
 		(property "Description" "Quad 2-input XOR"
-			(at 694.69 336.55 0)
+			(at 690.88 405.13 0)
 			(effects
 				(font

Commit message: almost done with ROM and SHM map
Parts:
- added D1, D2, D3, D4, D5, D6: D_Filled, symbol Device:D_Filled
Connections:
- net HH0: now also U15.13
- net at U1.11: now also U1.12, D1.1 (K), D2.1 (K), D3.1 (K), D4.1 (K), D5.1 (K), D6.1 (K)
- net at U1.13: now also U17.10
- net at U26.6: now also D3.2 (A)
- net at U17.6, U8.11 (LE): now also U1.5, U1.6
- net at U16.6: now also U17.9
- net at U20.11: now also D6.2 (A)
- net at U26.3: now also D4.2 (A)
- net at U16.12: now also U15.4
- net at U1.4: now also U15.5
- net at U27.12: now also D1.2 (A)
- net at U26.11: now also D2.2 (A)
- net at U15.11: now also U1.8, U1.9
- net at U15.12: now also U17.8, U3.10, U3.11
- net at U3.8: now also U16.10, U16.11, U16.9
- net at U3.9: now also U19.3
- net at U19.2: no longer U14.11
- net at U17.12: now also U12.6
- net at U17.13: now also U15.6
- net at U2.12: now also D5.2 (A)
- net at U19.6: no longer U16.9
Other:
- note added: "OS CHIP SELECT Only 0 if 1000-0011-0000-0001 > 1100-0001-1000-0000"
- note added: "Only 1 if OS, SCM, CS, RAND, and I/O is high(false)"
- moved on the sheet: U14D, U15B, U15D, U16C, U17B, U19A, U19B, U1B, U1C, U1D, U3C

Commit message: FINISHED MEMORY LOGICgit add .git add .!
Parts:
- added U30, U31, U32, U33, U34, U35, U36, U37, U38, U39, U40, U41, U42, U43, U44, U45: CY62256-70PC(RAM), Package_DIP:DIP-28_W15.24mm, symbol Memory_RAM:CY62256-70PC
Connections:
- net +5V: now also U29.14 (VCC)
- net A14: now also U19.2
- net A15: now also U19.1
- net GND: now also U29.7 (GND)
- net M15: no longer U27.9
- net at U13.2, U5.8: now also U13.9
- net at U3.9: now also U27.8; no longer U19.3
- new net: U19.3, U27.9
Other:
- note added: "ROM CHIP SELECT Only 0 if (0001-1111)-xxxx-xxxx-xxxx AND OS, SCM, CS RAND, I/O is false"
- note added: "SHARED MEM SELECT Only 0 if 0000-xxxx-xxxx-xxxx AND OS, SCM, CS, RAND, I/O is false"
- moved on the sheet: U14D, U19A, U27D, U29B

Commit message: Worked on the BANK
Parts:
- added U46: 74LS245, symbol 74xx:74LS245
Connections:
- net +5V: now also U46.20 (VCC)
- net A0: now also U30.10 (A0), U31.10 (A0), U32.10 (A0), U33.10 (A0), U34.10 (A0), U35.10 (A0), U36.10 (A0), U37.10 (A0), U38.10 (A0), U39.10 (A0), U40.10 (A0), U41.10 (A0), U42.10 (A0), U43.10 (A0), U44.10 (A0), U45.10 (A0)
- net A1: now also U30.9 (A1), U31.9 (A1), U32.9 (A1), U33.9 (A1), U34.9 (A1), U35.9 (A1), U36.9 (A1), U37.9 (A1), U38.9 (A1), U39.9 (A1), U40.9 (A1), U41.9 (A1), U42.9 (A1), U43.9 (A1), U44.9 (A1), U45.9 (A1)
- net A10: now also U30.21 (A10), U31.21 (A10), U32.21 (A10), U33.21 (A10), U34.21 (A10), U35.21 (A10), U36.21 (A10), U37.21 (A10), U38.21 (A10), U39.21 (A10), U40.21 (A10), U41.21 (A10), U42.21 (A10), U43.21 (A10), U44.21 (A10), U45.21 (A10)
- net A11: now also U30.23 (A11), U31.23 (A11), U32.23 (A11), U33.23 (A11), U34.23 (A11), U35.23 (A11), U36.23 (A11), U37.23 (A11), U38.23 (A11), U39.23 (A11), U40.23 (A11), U41.23 (A11), U42.23 (A11), U43.23 (A11), U44.23 (A11), U45.23 (A11)
- net A12: now also U30.2 (A12), U31.2 (A12), U32.2 (A12), U33.2 (A12), U34.2 (A12), U35.2 (A12), U36.2 (A12), U37.2 (A12), U38.2 (A12), U39.2 (A12), U40.2 (A12), U41.2 (A12), U42.2 (A12), U43.2 (A12), U44.2 (A12), U45.2 (A12)
- net A13: now also U30.26 (A13), U31.26 (A13), U32.26 (A13), U33.26 (A13), U34.26 (A13), U35.26 (A13), U36.26 (A13), U37.26 (A13), U38.26 (A13), U39.26 (A13), U40.26 (A13), U41.26 (A13), U42.26 (A13), U43.26 (A13), U44.26 (A13), U45.26 (A13)
- net A14: now also U30.1 (A14), U31.1 (A14), U32.1 (A14), U33.1 (A14), U34.1 (A14), U35.1 (A14), U36.1 (A14), U37.1 (A14), U38.1 (A14), U39.1 (A14), U40.1 (A14), U41.1 (A14), U42.1 (A14), U43.1 (A14), U44.1 (A14), U45.1 (A14)
- net A2: now also U30.8 (A2), U31.8 (A2), U32.8 (A2), U33.8 (A2), U34.8 (A2), U35.8 (A2), U36.8 (A2), U37.8 (A2), U38.8 (A2), U39.8 (A2), U40.8 (A2), U41.8 (A2), U42.8 (A2), U43.8 (A2), U44.8 (A2), U45.8 (A2)
- net A3: now also U30.7 (A3), U31.7 (A3), U32.7 (A3), U33.7 (A3), U34.7 (A3), U35.7 (A3), U36.7 (A3), U37.7 (A3), U38.7 (A3), U39.7 (A3), U40.7 (A3), U41.7 (A3), U42.7 (A3), U43.7 (A3), U44.7 (A3), U45.7 (A3)
- net A4: now also U30.6 (A4), U31.6 (A4), U32.6 (A4), U33.6 (A4), U34.6 (A4), U35.6 (A4), U36.6 (A4), U37.6 (A4), U38.6 (A4), U39.6 (A4), U40.6 (A4), U41.6 (A4), U42.6 (A4), U43.6 (A4), U44.6 (A4), U45.6 (A4)
- net A5: now also U30.5 (A5), U31.5 (A5), U32.5 (A5), U33.5 (A5), U34.5 (A5), U35.5 (A5), U36.5 (A5), U37.5 (A5), U38.5 (A5), U39.5 (A5), U40.5 (A5), U41.5 (A5), U42.5 (A5), U43.5 (A5), U44.5 (A5), U45.5 (A5)
- net A6: now also U30.4 (A6), U31.4 (A6), U32.4 (A6), U33.4 (A6), U34.4 (A6), U35.4 (A6), U36.4 (A6), U37.4 (A6), U38.4 (A6), U39.4 (A6), U40.4 (A6), U41.4 (A6), U42.4 (A6), U43.4 (A6), U44.4 (A6), U45.4 (A6)
- net A7: now also U30.3 (A7), U31.3 (A7), U32.3 (A7), U33.3 (A7), U34.3 (A7), U35.3 (A7), U36.3 (A7), U37.3 (A7), U38.3 (A7), U39.3 (A7), U40.3 (A7), U41.3 (A7), U42.3 (A7), U43.3 (A7), U44.3 (A7), U45.3 (A7)
- net A8: now also U30.25 (A8), U31.25 (A8), U32.25 (A8), U33.25 (A8), U34.25 (A8), U35.25 (A8), U36.25 (A8), U37.25 (A8), U38.25 (A8), U39.25 (A8), U40.25 (A8), U41.25 (A8), U42.25 (A8), U43.25 (A8), U44.25 (A8), U45.25 (A8)
- net A9: now also U30.24 (A9), U31.24 (A9), U32.24 (A9), U33.24 (A9), U34.24 (A9), U35.24 (A9), U36.24 (A9), U37.24 (A9), U38.24 (A9), U39.24 (A9), U40.24 (A9), U41.24 (A9), U42.24 (A9), U43.24 (A9), U44.24 (A9), U45.24 (A9)
- net C0: now also U30.20 (~{CS})
- net C1: now also U31.20 (~{CS})
- net C10: now also U40.20 (~{CS})
- net C11: now also U41.20 (~{CS})
- net C12: now also U42.20 (~{CS})
- net C13: now also U43.20 (~{CS})
- net C14: now also U44.20 (~{CS})
- net C15: now also U45.20 (~{CS})
- net C2: now also U32.20 (~{CS})
- net C3: now also U33.20 (~{CS})
- net C4: now also U34.20 (~{CS})
- net C5: now also U35.20 (~{CS})
- net C6: now also U36.20 (~{CS})
- net C7: now also U37.20 (~{CS})
- net C8: now also U38.20 (~{CS})
- net C9: now also U39.20 (~{CS})
- net D0: now also U46.18 (B0)
- net D1: now also U46.17 (B1)
- net D2: now also U46.16 (B2)
- net D3: now also U46.15 (B3)
- net D4: now also U46.14 (B4)
- net D5: now also U46.13 (B5)
- net D6: now also U46.12 (B6)
- net D7: now also U46.11 (B7)
- net GND: now also U46.10 (GND)
- net RW: now also U30.27 (~{WE}), U31.27 (~{WE}), U32.27 (~{WE}), U33.27 (~{WE}), U34.27 (~{WE}), U35.27 (~{WE}), U36.27 (~{WE}), U37.27 (~{WE}), U38.27 (~{WE}), U39.27 (~{WE}), U40.27 (~{WE}), U41.27 (~{WE}), U42.27 (~{WE}), U43.27 (~{WE}), U44.27 (~{WE}), U45.27 (~{WE}), U46.1 (A->B)
- net OS: now reaches U1.13, U17.10
- net BANKPICKER: now reaches U1.5, U1.6, U17.6, U8.11 (LE)
- net BANKMEM: now reaches U16.6, U17.9
- net BANKMEM: now also U46.19 (CE)
- net DD0: now reaches U35.11 (Q0)
- net DD0: now also U30.11 (Q0), U31.11 (Q0), U32.11 (Q0), U33.11 (Q0), U34.11 (Q0), U36.11 (Q0), U37.11 (Q0), U38.11 (Q0), U39.11 (Q0), U40.11 (Q0), U41.11 (Q0), U42.11 (Q0), U43.11 (Q0), U44.11 (Q0), U45.11 (Q0), U46.2 (A0)
- net DD1: now reaches U35.12 (Q1)
- net DD1: now also U30.12 (Q1), U31.12 (Q1), U32.12 (Q1), U33.12 (Q1), U34.12 (Q1), U36.12 (Q1), U37.12 (Q1), U38.12 (Q1), U39.12 (Q1), U40.12 (Q1), U41.12 (Q1), U42.12 (Q1), U43.12 (Q1), U44.12 (Q1), U45.12 (Q1), U46.3 (A1)
- net DD2: now reaches U35.13 (Q2)
- net DD2: now also U30.13 (Q2), U31.13 (Q2), U32.13 (Q2), U33.13 (Q2), U34.13 (Q2), U36.13 (Q2), U37.13 (Q2), U38.13 (Q2), U39.13 (Q2), U40.13 (Q2), U41.13 (Q2), U42.13 (Q2), U43.13 (Q2), U44.13 (Q2), U45.13 (Q2), U46.4 (A2)
- net at U35.14 (GND): now also U30.14 (GND), U31.14 (GND), U32.14 (GND), U33.14 (GND), U34.14 (GND), U36.14 (GND), U37.14 (GND), U38.14 (GND), U39.14 (GND), U40.14 (GND), U41.14 (GND), U42.14 (GND), U43.14 (GND), U44.14 (GND), U45.14 (GND)
- net DD3: now reaches U35.15 (Q3)
- net DD3: now also U30.15 (Q3), U31.15 (Q3), U32.15 (Q3), U33.15 (Q3), U34.15 (Q3), U36.15 (Q3), U37.15 (Q3), U38.15 (Q3), U39.15 (Q3), U40.15 (Q3), U41.15 (Q3), U42.15 (Q3), U43.15 (Q3), U44.15 (Q3), U45.15 (Q3), U46.5 (A3)
- net DD4: now reaches U35.16 (Q4)
- net DD4: now also U30.16 (Q4), U31.16 (Q4), U32.16 (Q4), U33.16 (Q4), U34.16 (Q4), U36.16 (Q4), U37.16 (Q4), U38.16 (Q4), U39.16 (Q4), U40.16 (Q4), U41.16 (Q4), U42.16 (Q4), U43.16 (Q4), U44.16 (Q4), U45.16 (Q4), U46.6 (A4)
- net DD5: now reaches U35.17 (Q5)
- net DD5: now also U30.17 (Q5), U31.17 (Q5), U32.17 (Q5), U33.17 (Q5), U34.17 (Q5), U36.17 (Q5), U37.17 (Q5), U38.17 (Q5), U39.17 (Q5), U40.17 (Q5), U41.17 (Q5), U42.17 (Q5), U43.17 (Q5), U44.17 (Q5), U45.17 (Q5), U46.7 (A5)
- net DD6: now reaches U35.18 (Q6)
- net DD6: now also U30.18 (Q6), U31.18 (Q6), U32.18 (Q6), U33.18 (Q6), U34.18 (Q6), U36.18 (Q6), U37.18 (Q6), U38.18 (Q6), U39.18 (Q6), U40.18 (Q6), U41.18 (Q6), U42.18 (Q6), U43.18 (Q6), U44.18 (Q6), U45.18 (Q6), U46.8 (A6)
- net DD7: now reaches U35.19 (Q7)
- net DD7: now also U30.19 (Q7), U31.19 (Q7), U32.19 (Q7), U33.19 (Q7), U34.19 (Q7), U36.19 (Q7), U37.19 (Q7), U38.19 (Q7), U39.19 (Q7), U40.19 (Q7), U41.19 (Q7), U42.19 (Q7), U43.19 (Q7), U44.19 (Q7), U45.19 (Q7), U46.9 (A7)
- net at U35.28 (VCC): now also U30.28 (VCC), U31.28 (VCC), U32.28 (VCC), U33.28 (VCC), U34.28 (VCC), U36.28 (VCC), U37.28 (VCC), U38.28 (VCC), U39.28 (VCC), U40.28 (VCC), U41.28 (VCC), U42.28 (VCC), U43.28 (VCC), U44.28 (VCC), U45.28 (VCC)
- net I_O: now reaches U15.4, U16.12
- net RAND: now reaches U12.6, U17.12
- net SHM: now reaches U16.8
- net ROM: now reaches U1.10
Other:
- moved on the sheet: U30, U31, U32, U33, U34, U35, U36, U37, U38, U39, U40, U41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

Commit message: Worked on the BANK
Connections:
- net +5V: now also U30.28 (VCC), U31.28 (VCC), U32.28 (VCC), U33.28 (VCC), U34.28 (VCC), U35.28 (VCC), U36.28 (VCC), U37.28 (VCC), U38.28 (VCC), U39.28 (VCC), U40.28 (VCC), U41.28 (VCC), U42.28 (VCC), U43.28 (VCC), U44.28 (VCC), U45.28 (VCC)
- net M0: now also U1.3
- net at U17.1, U27.6: no longer U4.1
- net ~{R}W: now reaches U35.22 (~{OE})
- net ~{R}W: now also U30.22 (~{OE}), U31.22 (~{OE}), U32.22 (~{OE}), U33.22 (~{OE}), U34.22 (~{OE}), U36.22 (~{OE}), U37.22 (~{OE}), U38.22 (~{OE}), U39.22 (~{OE}), U4.2, U40.22 (~{OE}), U41.22 (~{OE}), U42.22 (~{OE}), U43.22 (~{OE}), U44.22 (~{OE}), U45.22 (~{OE})
- net RW renamed R~{W}
- net R~{W}: now also U4.1
Other:
- moved on the sheet: U4A

Commit message: worked on mem bank
Parts:
- removed D1: SB140, symbol Device:D_Filled
- removed U2: 6522, Package_DIP:DIP-40_W15.24mm, symbol 6502:6522
Connections:
- net B0 is gone; now on net D0: DS1.7 (D0)
- net B1 is gone; now on net D1: DS1.8 (D1)
- net B2 is gone; now on net D2: DS1.9 (D2)
- net B3 is gone; now on net D3: DS1.10 (D3)
- net B4 is gone; now on net D4: DS1.11 (D4)
- net B5 is gone; now on net D5: DS1.12 (D5)
- net B6 is gone; now on net D6: DS1.13 (D6)
- net B7 is gone; now on net D7: DS1.14 (D7)
- net A0: no longer U5.13 (RS0)
- net A1: no longer U5.14 (RS1)
- net GND: no longer DS1.16 (LED(-)), RV1.1
- net IRQ: now also D2.1 (K); no longer D2.2 (A)
- net at U5.26 (~{IRQ}): now also D2.2 (A); no longer D2.1 (K)
- new net: DS1.16 (LED(-)), RV1.1
- no-connect marks 25 -> 16
Other:
- moved on the sheet: D2, DS1, RV1

Commit message: Made the Mem Bank work properly
Parts:
- removed U10: 74LS138, symbol 74xx_IEEE:74LS138
- removed U37, U38, U39, U40, U41, U42, U43, U44, U45: CY62256-70PC(RAM), Package_DIP:DIP-28_W15.24mm, symbol Memory_RAM:CY62256-70PC
Connections:
- net BANKMEM: now also U19.4
- net D6: no longer U9.6 (G1)
- net GND: now also U9.6 (G1)
- net R~{W}: now also U19.5, U19.6
Other:
- note added: "Only 0 if BANKMEM is selected and a Write is occuring from the CPU"
- moved on the sheet: U19B
